Commit message: added script to send joint commands with controller

File: zeus_arm/urdf/zeus_arm.urdf (robot description, URDF)
Before this commit: robot zeus_arm, 7 links, 6 joints
Links:
- link arm: geometry collision mesh filename=package://zeus_arm/meshes/arm.STL; visual mesh filename=package://zeus_arm/meshes/arm.STL
- link base_link: geometry collision mesh filename=package://zeus_arm/meshes/base_link.STL; visual mesh filename=package://zeus_arm/meshes/base_link.STL
- link base_plate: geometry collision mesh filename=package://zeus_arm/meshes/base_plate.STL; visual mesh filename=package://zeus_arm/meshes/base_plate.STL
- link forearm: geometry collision mesh filename=package://zeus_arm/meshes/forearm.STL; visual mesh filename=package://zeus_arm/meshes/forearm.STL
- link gripper: geometry collision mesh filename=package://zeus_arm/meshes/gripper.STL; visual mesh filename=package://zeus_arm/meshes/gripper.STL
- link wrist: geometry collision mesh filename=package://zeus_arm/meshes/wrist.STL; visual mesh filename=package://zeus_arm/meshes/wrist.STL
