Commit message: repo update, added arudino test code

File: zeus_arm/urdf/robot.urdf (robot description, URDF)
Before this commit: robot zeus_arm, 7 links, 6 joints
Joints:
- joint joint_2: limit lower=-0.174533 upper=1.91986 effort=20 velocity=3.19 -> lower=-1.57 upper=1.57 effort=20 velocity=3.19; origin xyz=-0.266 0.0881134 -0.113175 rpy=-1.5708 1.56905 -3.14159 -> xyz=-0.266 0.0881134 -0.113175 rpy=-1.5708 0 -3.14159

Commit message: update arm package

File: zeus_arm/urdf/robot.urdf (robot description, URDF)
Before this commit: robot zeus_arm, 7 links, 6 joints
Joints:
- joint joint_2: origin xyz=-0.266 0.0881134 -0.113175 rpy=-1.5708 0 -3.14159 -> xyz=-0.266 0.0881134 -0.113175 rpy=-1.5708 1.5708 -3.14159

Commit message: Added arm fail safe, calibration sequence, arduino code for new encoder and hall effect sensor, modified pins in arduino code, simulation code not final (tests still ongoing)

File: zeus_arm/urdf/robot.urdf (robot description, URDF)
Before this commit: robot zeus_arm, 7 links, 6 joints
Joints:
- joint joint_2: limit lower=-1.57 upper=1.57 effort=20 velocity=3.19 -> lower=-1.0 upper=1.57 effort=20 velocity=3.19

Commit message: Revert "Merge branch 'arm-jet-update'"
This reverts commit 3635869e71f27abe5f07b7dc301bff223cf1aca1, reversing
changes made to 54e90fbc9593c2a8f96bf9eabce9720e24dd27c7.

File: zeus_arm/urdf/robot.urdf (robot description, URDF)
Before this commit: robot zeus_arm, 7 links, 6 joints
Joints:
- joint joint_2: limit lower=-1.0 upper=1.57 effort=20 velocity=3.19 -> lower=-0.174533 upper=1.91986 effort=20 velocity=3.19; origin xyz=-0.266 0.0881134 -0.113175 rpy=-1.5708 1.5708 -3.14159 -> xyz=-0.266 0.0881134 -0.113175 rpy=-1.5708 1.56905 -3.14159
