Commit message: add rocker bogie as a spring

File: zeus_description/rover.urdf.xacro (robot description, xacro)
@@ -213,32 +213,55 @@
     </inertial>
   </link>
-  <joint name="rocker_right_joint" type="fixed">
+  <joint name="rocker_right_joint" type="revolute">
     <parent link="base_link"/>
     <child link="rocker_right"/>
     <origin rpy="0 -0.2 0" xyz="-0.3 -0.3 -0.4"/>
-    <!-- <axis xyz="0 1 0"/>
-    <dynamics damping="0.0" friction="10.0"/> -->
-  </joint>
-  <joint name="bogie_right_joint" type="continuous">
+    <limit  lower="-0.7854" upper="0.7854" effort="100000.0" velocity="10.0"/>
+    <axis xyz="0 1 0"/>
+		<joint_properties damping="0.5" friction="0.5"/>
+  </joint>
+  <transmission name="rocker_right_trans">
+    <type>transmission_interface/SimpleTransmission</type>
+    <joint name="rocker_right_joint">
+      <hardwareInterface>hardware_interface/EffortJointInterface</hardwareInterface>
+    </joint>
+    <actuator name="rocker_right_motor">
+      <hardwareInterface>hardware_interface/EffortJointInterface</hardwareInterface>
+      <mechanicalReduction>1</mechanicalReduction>
+    </actuator>
+  </transmission>
+  <joint name="bogie_right_joint" type="revolute">
     <parent link="rocker_right"/>
     <child link="bogie_right"/>
     <origin rpy="0 -0.5 0" xyz="0.35 0 -0.2"/>
     <axis xyz="0 1 0"/>
-    <dynamics damping="0.0" friction="10.0"/>
-  </joint>
-  <joint name="rocker_left_joint" type="fixed">
+    <dynamics damping="0.0" friction="100.0"/>
+    <limit  lower="-0.157075" upper="0.6" effort="100000.0" velocity="100000.0"/>
+  </joint>
+  <joint name="rocker_left_joint" type="continuous">
     <parent link="base_link"/>
     <child link="rocker_left"/>
     <origin rpy="0 -0.2 0" xyz="-0.3 0.3 -0.4"/>
-    <!-- <axis xyz="0 1 0"/>
-    <dynamics damping="0.0" friction="10.0"/>
-    <mimic joint="rocker_right_joint" multiplier="-1"/> -->
-  </joint>
-  <joint name="bogie_left_joint" type="continuous">
+    <limit  lower="-0.7854" upper="0.7854" effort="100000.0" velocity="10.0"/>
+    <axis xyz="0 1 0"/>
+		<joint_properties damping="0.5" friction="0.5"/>
+  </joint>
+  <transmission name="rocker_left_trans">
+    <type>transmission_interface/SimpleTransmission</type>
+    <joint name="rocker_left_joint">
+      <hardwareInterface>hardware_interface/EffortJointInterface</hardwareInterface>
+    </joint>
+    <actuator name="rocker_left_motor">
+      <hardwareInterface>hardware_interface/EffortJointInterface</hardwareInterface>
+      <mechanicalReduction>1</mechanicalReduction>
+    </actuator>
+  </transmission>
+  <joint name="bogie_left_joint" type="revolute">
     <parent link="rocker_left"/>
     <child link="bogie_left"/>
     <origin rpy="0 -0.5 0" xyz="0.35 0 -0.2"/>
     <axis xyz="0 1 0"/>
-    <dynamics damping="0.0" friction="10.0"/>
+    <dynamics damping="0.0" friction="100.0"/>
+    <limit  lower="-0.157075" upper="0.6" effort="100000.0" velocity="100000.0"/>
   </joint>
   <joint name="right_front_wheel_joint" type="continuous">
@@ -258,6 +281,6 @@
   </transmission>
   <gazebo reference="$right_front_wheel">
-    <mu1 value="0.5"/>
-    <mu2 value="0.5"/>
+    <mu1 value="0.1"/>
+    <mu2 value="0.1"/>
     <kp value="10000000.0" />
     <kd value="1.0" />
@@ -280,6 +303,6 @@
   </transmission>
   <gazebo reference="$right_middle_wheel">
-    <mu1 value="0.5"/>
-    <mu2 value="0.5"/>
+    <mu1 value="0.1"/>
+    <mu2 value="0.1"/>
     <kp value="10000000.0" />
     <kd value="1.0" />
@@ -302,6 +325,6 @@
   </transmission>
   <gazebo reference="$right_rear_wheel">
-    <mu1 value="0.5"/>
-    <mu2 value="0.5"/>
+    <mu1 value="0.1"/>
+    <mu2 value="0.1"/>
     <kp value="10000000.0" />
     <kd value="1.0" />
@@ -324,6 +347,6 @@
   </transmission>
   <gazebo reference="$left_front_wheel">
-    <mu1 value="0.5"/>
-    <mu2 value="0.5"/>
+    <mu1 value="0.1"/>
+    <mu2 value="0.1"/>
     <kp value="10000000.0" />
     <kd value="1.0" />
@@ -346,6 +369,6 @@
   </transmission>
   <gazebo reference="$left_middle_wheel">
-    <mu1 value="0.5"/>
-    <mu2 value="0.5"/>
+    <mu1 value="0.1"/>
+    <mu2 value="0.1"/>
     <kp value="10000000.0" />
     <kd value="1.0" />
@@ -368,6 +391,6 @@
   </transmission>
   <gazebo reference="$left_rear_wheel">
-    <mu1 value="0.5"/>
-    <mu2 value="0.5"/>
+    <mu1 value="0.1"/>
+    <mu2 value="0.1"/>
     <kp value="10000000.0" />
     <kd value="1.0" />

Commit message: add xacro to urdf, fix wheel non-slip problem, add camera and imu

File: zeus_description/rover.urdf.xacro (robot description, xacro)
@@ -1,26 +1,50 @@
 <?xml version="1.0"?>
-<robot name="myfirst">
-  <material name="gray">
-    <color rgba="0.5 0.5 0.5 1"/>
-  </material>
+<robot xmlns:xacro="http://www.ros.org/wiki/xacro" name="zeus">
+  <xacro:property name="deg90" value="1.57075" />
+  <xacro:property name="deg45" value="0.7854" />
+  <xacro:property name="frame_width" value="0.6" />
+  <xacro:property name="frame_height" value="0.3" />
+  <xacro:property name="frame_length" value="0.82" />
+  <xacro:property name="frame_mass" value="50" />
+  <xacro:property name="rocker_mass" value="10" />
+  <xacro:property name="bogie_mass" value="10" />
+  <xacro:property name="wheel_radius" value="0.1" />
+  <xacro:property name="wheel_width" value="0.1" />
+  <xacro:property name="wheel_mass" value="1" />
+  <xacro:property name="wheel_mu1" value="0.5" />
+  <xacro:property name="wheel_mu2" value="0.5" />
+  <xacro:property name="wheel_kp" value="10000000.0" />
+  <xacro:property name="wheel_kd" value="1" />
+  <!-- High level dummy link for ODE -->
   <link name="base_link">
+  </link>
+  <!-- Frame -->
+  <link name="frame_link">
     <visual>
       <geometry>
         <mesh filename="file://$(find zeus_description)/STL/Z1.stl"/>
       </geometry>
-      <origin rpy="1.57075 0 0" xyz="0 0 0"/>
-      <material name="gray"/>
-    </visual>
-    <collision>
-      <geometry>
-        <box size="0.82 0.6 0.3"/>
+      <origin rpy="${deg90} 0 0" xyz="0 0 0"/>
+    </visual>
+    <collision>
+      <geometry>
+        <box size="${frame_length} ${frame_width} ${frame_height}"/>
       </geometry>
       <origin rpy="0 0 0" xyz="-0.27 -0.02 -0.45"/>
     </collision>
     <inertial>
-      <mass value="50"/>
-      <inertia ixx="0.4" ixy="0.0" ixz="0.0" iyy="0.4" iyz="0.0" izz="0.4"/>
-    </inertial>
-  </link>
+      <mass value="${frame_mass}"/>
+      <inertia ixx="4" ixy="0.0" ixz="0.0" iyy="4" iyz="0.0" izz="4"/>
+    </inertial>
+  </link>
+  <joint name="frame_link_joint" type="fixed">
+    <parent link="base_link"/>
+    <child link="frame_link"/>
+    <origin rpy="0 -0 0" xyz="0 0 0"/>
+  </joint>
+  <gazebo reference="frame_link">
+    <material>Gazebo/DarkGray</material>
+  </gazebo>
+<!-- Rocker right -->
   <link name="rocker_right">
     <visual>
@@ -29,193 +53,15 @@
       </geometry>
       <origin rpy="0 0 0" xyz="0 0 0"/>
-      <material name="gray"/>
-    </visual>
-    <!-- <collision>
-      <geometry>
-        <mesh filename="file://$(find zeus_description)/STL/rocker_right.stl"/>
-      </geometry>
-      <origin rpy="0 0 0" xyz="-0 0 0"/>
-    </collision> -->
-    <inertial>
-      <mass value="10"/>
-      <inertia ixx="0.4" ixy="0.0" ixz="0.0" iyy="0.4" iyz="0.0" izz="0.4"/>
-    </inertial>
-  </link>
-  <link name="bogie_right">
-    <visual>
-      <geometry>
-        <mesh filename="file://$(find zeus_description)/STL/bogie.stl"/>
-      </geometry>
-      <origin rpy="0 0 0" xyz="0 0 0"/>
-      <material name="gray"/>
-    </visual>
-    <!-- <collision>
-      <geometry>
-        <mesh filename="file://$(find zeus_description)/STL/bogie.stl"/>
-      </geometry>
-      <origin rpy="0 0 0" xyz="0 0 0"/>
-    </collision> -->
-    <inertial>
-      <mass value="10"/>
-      <inertia ixx="0.4" ixy="0.0" ixz="0.0" iyy="0.4" iyz="0.0" izz="0.4"/>
-    </inertial>
-  </link>
-  <link name="rocker_left">
-    <visual>
-      <geometry>
-        <mesh filename="file://$(find zeus_description)/STL/rocker_right.stl"/>
-      </geometry>
-      <origin rpy="0 0 0" xyz="0 0 0"/>
-      <material name="gray"/>
-    </visual>
-    <!-- <collision>
-      <geometry>
-        <mesh filename="file://$(find zeus_description)/STL/rocker_right.stl"/>
-      </geometry>
-      <origin rpy="0 0 0" xyz="-0 0 0"/>
-    </collision> -->
-    <inertial>
-      <mass value="10"/>
-      <inertia ixx="0.4" ixy="0.0" ixz="0.0" iyy="0.4" iyz="0.0" izz="0.4"/>
-    </inertial>
-  </link>
-  <link name="bogie_left">
-    <visual>
-      <geometry>
-        <mesh filename="file://$(find zeus_description)/STL/bogie.stl"/>
-      </geometry>
-      <origin rpy="0 0 0" xyz="0 0 0"/>
-      <material name="gray"/>
-    </visual>
-    <!-- <collision>
-      <geometry>
-        <box size="1.3 0.75 1.3"/>
-      </geometry>
-      <origin rpy="0 0 0" xyz="0 0 0"/>
-    </collision> -->
-    <inertial>
-      <mass value="10"/>
-      <inertia ixx="0.4" ixy="0.0" ixz="0.0" iyy="0.4" iyz="0.0" izz="0.4"/>
-    </inertial>
-  </link>
-  <link name="right_front_wheel">
-    <visual>
-      <origin rpy="0 0 0" xyz="0 0 0"/>
-      <geometry>
-       <mesh filename="file://$(find zeus_description)/STL/Z1-PRP-01-001.stl"/>
-      </geometry>
-      <material name="black"/>
-    </visual>
-    <collision>
-      <geometry>
-        <cylinder length="0.1" radius="0.1"/>
-      </geometry>
-      <origin rpy="0 0 0" xyz="0 0 0"/>
-    </collision>
-    <inertial>
-      <mass value="1"/>
-      <inertia ixx="0.1" ixy="0.0" ixz="0.0" iyy="0.1" iyz="0.0" izz="0.1"/>
-    </inertial>
-  </link>
-  <link name="right_middle_wheel">
-    <visual>
-      <origin rpy="0 0 0" xyz="0 0 0"/>
-      <geometry>
-       <mesh filename="file://$(find zeus_description)/STL/Z1-PRP-01-001.stl"/>
-      </geometry>
-      <material name="black"/>
-    </visual>
-    <collision>
-      <geometry>
-        <cylinder length="0.1" radius="0.1"/>
-      </geometry>
-      <origin rpy="0 0 0" xyz="0 0 0"/>
-    </collision>
-    <inertial>
-      <mass value="1"/>
-      <inertia ixx="0.1" ixy="0.0" ixz="0.0" iyy="0.1" iyz="0.0" izz="0.1"/>
-    </inertial>
-  </link>
-  <link name="right_rear_wheel">
-    <visual>
-      <origin rpy="1.57075 0 0" xyz="0 0 0"/>
-      <geometry>
-        <mesh filename="file://$(find zeus_description)/STL/Z1-PRP-01-001.stl"/>
-      </geometry>
-      <material name="black"/>
-    </visual>
-    <collision>
-      <geometry>
-        <cylinder length="0.1" radius="0.1"/>
-      </geometry>
-      <origin rpy="1.57075 0 0" xyz="0 0 0"/>
-    </collision>
-    <inertial>
-      <mass value="1"/>
-      <inertia ixx="0.1" ixy="0.0" ixz="0.0" iyy="0.1" iyz="0.0" izz="0.1"/>
-    </inertial>
-  </link>
-  <link name="left_front_wheel">
-    <visual>
-      <origin rpy="0 0 0" xyz="0 0 0"/>
-      <geometry>
-       <mesh filename="file://$(find zeus_description)/STL/Z1-PRP-01-001.stl"/>
-      </geometry>
-      <material name="black"/>
-    </visual>
-    <collision>
-      <geometry>
-        <cylinder length="0.1" radius="0.1"/>
-      </geometry>
-      <origin rpy="0 0 0" xyz="0 0 0"/>
-    </collision>
-    <inertial>
-      <mass value="1"/>
-      <inertia ixx="0.1" ixy="0.0" ixz="0.0" iyy="0.1" iyz="0.0" izz="0.1"/>
-    </inertial>
-  </link>
-  <link name="left_middle_wheel">
-    <visual>
-      <origin rpy="0 0 0" xyz="0 0 0"/>
-      <geometry>
-       <mesh filename="file://$(find zeus_description)/STL/Z1-PRP-01-001.stl"/>
-      </geometry>
-      <material name="black"/>
-    </visual>
-    <collision>
-      <geometry>
-        <cylinder length="0.1" radius="0.1"/>
-      </geometry>
-      <origin rpy="0 0 0" xyz="0 0 0"/>
-    </collision>
-    <inertial>
-      <mass value="1"/>
-      <inertia ixx="0.1" ixy="0.0" ixz="0.0" iyy="0.1" iyz="0.0" izz="0.1"/>
-    </inertial>
-  </link>
-  <link name="left_rear_wheel">
-    <visual>
-      <origin rpy="1.57075 0 0" xyz="0 0 0"/>
-      <geometry>
-        <mesh filename="file://$(find zeus_description)/STL/Z1-PRP-01-001.stl"/>
-      </geometry>
-      <material name="black"/>
-    </visual>
-    <collision>
-      <geometry>
-        <cylinder length="0.1" radius="0.1"/>
-      </geometry>
-      <origin rpy="1.57075 0 0" xyz="0 0 0"/>
-    </collision>
-    <inertial>
-      <mass value="1"/>
-      <inertia ixx="0.1" ixy="0.0" ixz="0.0" iyy="0.1" iyz="0.0" izz="0.1"/>
+    </visual>
+    <inertial>
+      <mass value="${rocker_mass}"/>
+      <inertia ixx="${wheel_mass*wheel_radius*wheel_radius}" ixy="0.0" ixz="0.0" iyy="${wheel_mass*wheel_radius*wheel_radius}" iyz="0.0" izz="${wheel_mass*wheel_radius*wheel_radius}"/>
     </inertial>
   </link>
   <joint name="rocker_right_joint" type="revolute">
-    <parent link="base_link"/>
+    <parent link="frame_link"/>
     <child link="rocker_right"/>
     <origin rpy="0 -0.2 0" xyz="-0.3 -0.3 -0.4"/>
-    <limit  lower="-0.7854" upper="0.7854" effort="100000.0" velocity="10.0"/>
+    <limit  lower="${-deg45}" upper="${deg45}" effort="100000.0" velocity="10.0"/>
     <axis xyz="0 1 0"/>
 		<joint_properties damping="0.5" friction="0.5"/>
@@ -231,4 +77,21 @@
     </actuator>
   </transmission>
+  <gazebo reference="rocker_right">
+    <material>Gazebo/Gray</material>
+  </gazebo>
+  <!-- Bogie right -->
+  <link name="bogie_right">
+    <visual>
+      <geometry>
+        <mesh filename="file://$(find zeus_description)/STL/bogie.stl"/>
+      </geometry>
+      <origin rpy="0 0 0" xyz="0 0 0"/>
+      <material name="gray"/>
+    </visual>
+    <inertial>
+      <mass value="${bogie_mass}"/>
+      <inertia ixx="0.01" ixy="0.0" ixz="0.0" iyy="0.01" iyz="0.0" izz="0.01"/>
+    </inertial>
+  </link>
   <joint name="bogie_right_joint" type="revolute">
     <parent link="rocker_right"/>
@@ -236,12 +99,29 @@
     <origin rpy="0 -0.5 0" xyz="0.35 0 -0.2"/>
     <axis xyz="0 1 0"/>
-    <dynamics damping="0.0" friction="100.0"/>
-    <limit  lower="-0.157075" upper="0.6" effort="100000.0" velocity="100000.0"/>
-  </joint>
+    <dynamics damping="0.0" friction="10.0"/>
+    <limit  lower="${-deg90}" upper="0.6" effort="100000.0" velocity="100000.0"/>
+  </joint>
+  <gazebo reference="bogie_right">
+    <material>Gazebo/Gray</material>
+  </gazebo>
+  <!-- Rocker left -->
+  <link name="rocker_left">
+    <visual>
+      <geometry>
+        <mesh filename="file://$(find zeus_description)/STL/rocker_left.stl"/>
+      </geometry>
+      <origin rpy="0 0 0" xyz="0 0 0"/>
+      <material name="gray"/>
+    </visual>
+    <inertial>
+      <mass value="${rocker_mass}"/>
+      <inertia ixx="0.01" ixy="0.0" ixz="0.0" iyy="0.01" iyz="0.0" izz="0.01"/>
+    </inertial>
+  </link>
   <joint name="rocker_left_joint" type="continuous">
-    <parent link="base_link"/>
+    <parent link="frame_link"/>
     <child link="rocker_left"/>
     <origin rpy="0 -0.2 0" xyz="-0.3 0.3 -0.4"/>
-    <limit  lower="-0.7854" upper="0.7854" effort="100000.0" velocity="10.0"/>
+    <limit  lower="${-deg45}" upper="${deg45}" effort="100000.0" velocity="10.0"/>
     <axis xyz="0 1 0"/>
 		<joint_properties damping="0.5" friction="0.5"/>
@@ -257,4 +137,21 @@
     </actuator>
   </transmission>
+  <gazebo reference="rocker_left">
+    <material>Gazebo/Gray</material>
+  </gazebo>
+  <!-- Bogie left -->
+  <link name="bogie_left">
+    <visual>
+      <geometry>
+        <mesh filename="file://$(find zeus_description)/STL/bogie.stl"/>
+      </geometry>
+      <origin rpy="0 0 0" xyz="0 0 0"/>
+      <material name="gray"/>
+    </visual>
+    <inertial>
+      <mass value="${bogie_mass}"/>
+      <inertia ixx="0.01" ixy="0.0" ixz="0.0" iyy="0.01" iyz="0.0" izz="0.01"/>
+    </inertial>
+  </link>
   <joint name="bogie_left_joint" type="revolute">
     <parent link="rocker_left"/>
@@ -262,11 +159,33 @@
     <origin rpy="0 -0.5 0" xyz="0.35 0 -0.2"/>
     <axis xyz="0 1 0"/>
-    <dynamics damping="0.0" friction="100.0"/>
-    <limit  lower="-0.157075" upper="0.6" effort="100000.0" velocity="100000.0"/>
-  </joint>
+    <dynamics damping="0.0" friction="10.0"/>
+    <limit  lower="${-deg90}" upper="0.6" effort="100000.0" velocity="100000.0"/>
+  </joint>
+  <gazebo reference="bogie_left">
+    <material>Gazebo/Gray</material>
+  </gazebo>
+  <!-- Wheel front right -->
+  <link name="right_front_wheel">
+    <visual>
+      <origin rpy="0 0 0" xyz="0 0 0"/>
+      <geometry>
+       <mesh filename="file://$(find zeus_description)/STL/Z1-PRP-01-001.stl"/>
+      </geometry>
+    </visual>
+    <collision>
+      <geometry>
+        <cylinder length="${wheel_width}" radius="${wheel_radius}"/>
+      </geometry>
+      <origin rpy="0 0 0" xyz="0 0 0"/>
+    </collision>
+    <inertial>
+      <mass value="${wheel_mass}"/>
+      <inertia ixx="${wheel_mass*wheel_radius*wheel_radius}" ixy="0.0" ixz="0.0" iyy="${wheel_mass*wheel_radius*wheel_radius}" iyz="0.0" izz="${wheel_mass*wheel_radius*wheel_radius}"/>
+    </inertial>
+  </link>
   <joint name="right_front_wheel_joint" type="continuous">
     <parent link="bogie_right"/>
     <child link="right_front_wheel"/>
-   <origin rpy="1.57075 0 0" xyz="0 -0.05 -0.45"/>
+   <origin rpy="${deg90} 0 0" xyz="0 -0.05 -0.45"/>
     <axis xyz="0 0 -1"/>
   </joint>
@@ -280,15 +199,35 @@
     </joint>
   </transmission>
-  <gazebo reference="$right_front_wheel">
-    <mu1 value="0.1"/>
-    <mu2 value="0.1"/>
-    <kp value="10000000.0" />
-    <kd value="1.0" />
-    <material>Gazebo/Grey</material>
-  </gazebo>
+  <gazebo reference="right_front_wheel">
+    <mu1 value="${wheel_mu1}"/>
+    <mu2 value="${wheel_mu2}"/>
+    <kp value="${wheel_kp}" />
+    <kd value="${wheel_kd}" />
+    <material>Gazebo/Black</material>
+  </gazebo>
+  <!-- Wheel middle right -->
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
Commit message: added stereo camera to sim

File: zeus_description/rover.urdf.xacro (robot description, xacro)
@@ -535,5 +535,6 @@
     <plugin name="gps_controller" filename="libhector_gazebo_ros_gps.so">
       <robotNamespace>zeus</robotNamespace>
-      <updateRate>1</updateRate>
+      <alwayson>true</alwayson>
+      <updateRate>1.0</updateRate>
       <bodyName>base_link</bodyName>
       <frameId>base_link</frameId>
@@ -548,5 +549,31 @@
   </gazebo>
   <!-- Stereo camera -->
-  <!-- <gazebo reference="left_camera_frame">
+  <link name="stereo_link">
+    <collision>
+      <origin xyz="0 0 0" rpy="0 0 0"/>
+      <geometry>
+    <box size="0.05 0.05 0.05"/>
+      </geometry>
+    </collision>
+    <visual>
+      <origin xyz="0 0 0" rpy="0 0 0"/>
+      <geometry>
+    <box size="0.05 0.05 0.01"/>
+      </geometry>
+    </visual>
+    <inertial>
+      <mass value="1e-5" />
+      <origin xyz="0 0 0" rpy="0 0 0"/>
+      <inertia ixx="1e-6" ixy="0" ixz="0" iyy="1e-6" iyz="0" izz="1e-6" />
+    </inertial>
+  </link>
+  <joint name="stereo_link" type="fixed">
+    <axis xyz="0 1 0" />
+    <origin xyz="0.13 -0.02 -0.29" rpy="0 0 0"/>
+    <parent link="frame_link"/>
+    <child link="stereo_link"/>
+  </joint>
+  <!-- Simple Stereo camera -->
+  <!--<gazebo reference="stereo_link">
     <sensor type="multicamera" name="stereo_camera">
       <update_rate>30.0</update_rate>
@@ -589,5 +616,5 @@
         <alwaysOn>true</alwaysOn>
         <updateRate>0.0</updateRate>
-        <cameraName>multisense_sl/camera</cameraName>
+        <cameraName>zed</cameraName>
         <imageTopicName>image_raw</imageTopicName>
         <cameraInfoTopicName>camera_info</cameraInfoTopicName>
@@ -602,4 +629,46 @@
     </sensor>
   </gazebo> -->
+  <!-- Stereo camera with depth -->
+  <gazebo reference="stereo_link">
+  <sensor name="stereo_depth_camera" type="depth">
+    <update_rate>20</update_rate>
+    <camera>
+      <horizontal_fov>1.047198</horizontal_fov>
+      <image>
+        <width>640</width>
+        <height>480</height>
+        <format>R8G8B8</format>
+      </image>
+      <clip>
+        <near>0.05</near>
+        <far>3</far>
+      </clip>
+    </camera>
+    <plugin name="stereo_depth_controller" filename="libgazebo_ros_openni_kinect.so">
+      <baseline>0.2</baseline>
+      <alwaysOn>true</alwaysOn>
+      <updateRate>1.0</updateRate>
+      <cameraName>zed</cameraName>
+      <imageTopicName>/zed/color/image_raw</imageTopicName>
+      <cameraInfoTopicName>/zed/color/camera_info</cameraInfoTopicName>
+      <depthImageTopicName>/zed/depth/image_raw</depthImageTopicName>
+      <depthImageInfoTopicName>/zed/depth/camera_info</depthImageInfoTopicName>
+      <pointCloudTopicName>/zed/depth/points</pointCloudTopicName>
+      <frameName>stereo_link</frameName>
+      <pointCloudCutoff>0.5</pointCloudCutoff>
+      <pointCloudCutoffMax>3.0</pointCloudCutoffMax>
+      <distortionK1>0.00000001</distortionK1>
+      <distortionK2>0.00000001</distortionK2>
+      <distortionK3>0.00000001</distortionK3>
+      <distortionT1>0.00000001</distortionT1>
+      <distortionT2>0.00000001</distortionT2>
+      <CxPrime>0</CxPrime>
+      <Cx>0</Cx>
+      <Cy>0</Cy>
+      <focalLength>0</focalLength>
+      <hackBaseline>0</hackBaseline>
+    </plugin>
+  </sensor>
+  </gazebo>
   <!-- Controllers -->
   <gazebo>

Commit message: changed mars env terrain

File: zeus_description/rover.urdf.xacro (robot description, xacro)
@@ -12,6 +12,6 @@
   <xacro:property name="wheel_width" value="0.1" />
   <xacro:property name="wheel_mass" value="1" />
-  <xacro:property name="wheel_mu1" value="0.5" />
-  <xacro:property name="wheel_mu2" value="0.5" />
+  <xacro:property name="wheel_mu1" value="0.2" />
+  <xacro:property name="wheel_mu2" value="3.0" />
   <xacro:property name="wheel_kp" value="10000000.0" />
   <xacro:property name="wheel_kd" value="1" />

Commit message: added launch files, working on move base setup

File: zeus_description/rover.urdf.xacro (robot description, xacro)
@@ -568,8 +568,8 @@
     </inertial>
   </link>
-  <joint name="stereo_link" type="fixed">
+  <joint name="stereo_joint" type="fixed">
     <axis xyz="0 1 0" />
     <origin xyz="0.13 -0.02 -0.29" rpy="0 0 0"/>
-    <parent link="frame_link"/>
+    <parent link="base_link"/>
     <child link="stereo_link"/>
   </joint>
