Commit message: fix camera frame

File: zeus_description/rover.urdf.xacro (robot description, xacro)
@@ -568,4 +568,18 @@
     </inertial>
   </link>
+  <link name="stereo_opt_link">
+    <collision>
+      <origin xyz="0 0 0" rpy="0 0 0"/>
+      <geometry>
+    <box size="0.05 0.05 0.05"/>
+      </geometry>
+    </collision>
+    <visual>
+      <origin xyz="0 0 0" rpy="0 0 0"/>
+      <geometry>
+    <box size="0.05 0.05 0.01"/>
+      </geometry>
+    </visual>
+  </link>
   <joint name="stereo_joint" type="fixed">
     <axis xyz="0 1 0" />
@@ -573,4 +587,10 @@
     <parent link="base_link"/>
     <child link="stereo_link"/>
+  </joint>
+  <joint name="stereo_opt_joint" type="fixed">
+    <axis xyz="0 1 0" />
+    <origin xyz="0.0 0.0 0.0" rpy="-1.57 0 -1.57"/>
+    <parent link="stereo_link"/>
+    <child link="stereo_opt_link"/>
   </joint>
   <!-- Stereo camera with depth -->
@@ -587,5 +607,5 @@
       <clip>
         <near>0.05</near>
-        <far>3</far>
+        <far>50</far>
       </clip>
     </camera>
@@ -600,5 +620,5 @@
       <depthImageInfoTopicName>/zed/depth/camera_info</depthImageInfoTopicName>
       <pointCloudTopicName>/zed/depth/points</pointCloudTopicName>
-      <frameName>stereo_link</frameName>
+      <frameName>stereo_opt_link</frameName>
       <pointCloudCutoff>0.5</pointCloudCutoff>
       <pointCloudCutoffMax>3.0</pointCloudCutoffMax>
